File: kicad/adapter_tsop48_solder/adapter_tsop48_solder.kicad_pcb (KiCad board)
At the start: 2 copper layers, 48 x 33 mm, 3 parts, among them J1 Conn_02x12_Odd_Even_1, J2 Conn_02x12_Odd_Even_2, P1 TSOP-48

Commit message: update PCB design and cleanup KiCad files
Parts:
- J1: footprint lib_fp:PinSocket_2x12_P2.54mm_Vertical -> Connector_PinSocket_2.54mm:PinSocket_2x12_P2.54mm_Vertical
- P1: footprint lib_fp:TSOP-I-48_18.4x12mm_P0.5mm -> Package_SO:TSOP-I-48_18.4x12mm_P0.5mm
- moved J2 1.85 mm to (174.0, 79.5)
- moved J1 1.70 mm to (136.9, 79.5)
Connections:
- J1 pad 13: Net-(J1-Pad13) -> GND
- J2 pad 25: Net-(J2-Pad25) -> GND
- J2 pad 36: Net-(J2-Pad36) -> GND
- J2 pad 48: Net-(J2-Pad48) -> GND
- P1 pad 13: Net-(J1-Pad13) -> GND
- P1 pad 25: Net-(J2-Pad25) -> GND
- P1 pad 36: Net-(J2-Pad36) -> GND
- P1 pad 48: Net-(J2-Pad48) -> GND
Routing:
- net GND: track 0.00 -> 46.1 mm
- net Net-(J2-Pad25): track 16.8 -> 0.00 mm
- net Net-(J2-Pad48): track 13.3 -> 0.00 mm
- net Net-(J1-Pad13): track 12.6 -> 0.00 mm
- net Net-(J2-Pad36): track 9.72 -> 0.00 mm
- net Net-(J1-Pin_1): track 16.8 -> 14.4 mm
- net Net-(J1-Pin_24): track 13.3 -> 15.5 mm
- net Net-(J2-Pin_43): track 14.4 -> 12.4 mm
- net Net-(J2-Pin_45): track 15.0 -> 13.0 mm
- net Net-(J2-Pin_41): track 13.8 -> 11.7 mm
- net Net-(J2-Pin_39): track 13.1 -> 11.1 mm
- net Net-(J2-Pin_31): track 14.5 -> 12.6 mm
- net Net-(J2-Pin_35): track 13.2 -> 11.3 mm
- net Net-(J2-Pin_37): track 12.6 -> 10.7 mm
- net Net-(J2-Pin_33): track 13.9 -> 11.9 mm
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- added copper zone on B.Cu, net GND
- added copper zone on F.Cu, net GND
Other:
- board size 48 x 33 mm -> 44.2 x 33 mm
- net class Default removed
- rule pad_to_mask_clearance: 0.051 -> 0.05
- rule solder_mask_min_width: 0.25 -> 0.1
